Commit message: URDF loading working

File: SOFTWARE/little_red_rover_ws/src/little_red_rover/assets/rover/robot.urdf (robot description, URDF)
Before this commit: robot onshape, 3 links, 2 joints
Links:
- added link base_link
- link robot_body: geometry collision mesh filename=http://localhost:8100/rover/lidar_motor.stl; collision mesh filename=http://localhost:8100/rover/lidar_top.stl
- link wheel: geometry collision mesh filename=http://localhost:8100/rover/wheel.stl; visual mesh filename=http://localhost:8100/rover/wheel_visual.stl
- link wheel_2: geometry collision mesh filename=http://localhost:8100/rover/wheel.stl; visual mesh filename=http://localhost:8100/rover/wheel_2_visual.stl
Joints:
- added joint base_link_to_base: type fixed, parent base_link, child robot_body, origin xyz=0 0 0 rpy=0.0 0 0
