File: HARDWARE/little_red_rover/little_red_rover.kicad_sch (KiCad schematic)
At the start: 61 parts, among them J1 USB_C_Receptacle_USB2.0_14P, J2 Conn_01x04_Socket, J5 Conn_01x01_Socket, J6 Conn_01x01_Socket, J7 Conn_01x06, J8 Conn_02x12_Odd_Even, J9 Conn_01x06, Q1 PMOS, Q2 PMOS, SW1 SW_Push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

Commit message: Change battery IC for a higher current version, change motors to be powered straight from charger output rather than 5v regulation.
Parts:
- removed U2: BQ24230RGT, Package_DFN_QFN:VQFN-16-1EP_3x3mm_P0.5mm_EP1.68x1.68mm_ThermalVias, symbol Power_Management:BQ24230RGT
- added C16: 22uF, Capacitor_SMD:C_0603_1608Metric_Pad1.08x0.95mm_HandSolder, symbol Device:C
- added U2: BQ24072RGT, Package_DFN_QFN:VQFN-16-1EP_3x3mm_P0.5mm_EP1.6x1.6mm, symbol Battery_Management:BQ24072RGT
- C2: value 4.7uF -> 47uF
- C7, C8: value 10uF -> 22uF
Connections:
- net +5V: now also C16.1; no longer C7.1, C8.1, U5.1 (VM), U6.1 (VM)
- net +BATT: now also C5.2, U2.2 (BAT), U2.3 (BAT); no longer C5.1, SW4.1 (A)
- net CHG: now also U2.9 (~{CHG})
- net GND: now also C1.1, C2.1, C5.1, C16.2, U2.15 (TD), U2.17 (VSS), U2.4 (~{CE}), U2.6 (EN1), U2.8 (VSS); no longer C1.2, C2.2, C5.2
- net ILIM: now also U2.12 (ILIM)
- net ISET: now also U2.16 (ISET)
- net PGOOD: now also U2.7 (~{PGOOD})
- net TMR: now also U2.14 (TMR)
- net TS: now also U2.1 (TS)
- net VDD: now also C7.1, C8.1, U5.1 (VM), U6.1 (VM)
- net charger_out: now also C2.2, SW4.1 (A), U2.10 (OUT), U2.11 (OUT), U2.5 (EN2); no longer C2.1
- net usb_5v: now also C1.2, U2.13 (IN); no longer C1.1
Other:
- moved on the sheet: C11, C12, C13, C14, C15, C3, C4, C6, D3, D4, D5, D7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

Commit message: Ordered PCB v0.2.2: FA '24 beta test
Parts:
- added R20, R8: 10k, Resistor_SMD:R_0603_1608Metric_Pad0.98x0.95mm_HandSolder, symbol Device:R
- added R7: 47k, Resistor_SMD:R_0603_1608Metric_Pad0.98x0.95mm_HandSolder, symbol Device:R
- R10: value 47k -> 33k
- R11: value 47k -> 1k
Connections:
- net +3.3V: now also R20.1
- net +5V: now also J8.19 (Pin_19)
- net GND: now also R7.1; no longer J8.4 (Pin_4)
- net GPIO_16: now also J8.5 (Pin_5); no longer J8.6 (Pin_6)
- net GPIO_21: now also J8.7 (Pin_7); no longer J8.5 (Pin_5)
- net GPIO_33: now also J8.9 (Pin_9); no longer J8.8 (Pin_8)
- net GPIO_34: now also J8.11 (Pin_11); no longer J8.7 (Pin_7)
- net GPIO_35: now also J8.13 (Pin_13); no longer J8.10 (Pin_10)
- net GPIO_36: now also J8.15 (Pin_15); no longer J8.9 (Pin_9)
- net GPIO_37: now also J8.17 (Pin_17); no longer J8.12 (Pin_12)
- net GPIO_38: now also J8.4 (Pin_4); no longer J8.11 (Pin_11)
- net GPIO_39: now also J8.6 (Pin_6); no longer J8.14 (Pin_14)
- net GPIO_40: now also J8.8 (Pin_8); no longer J8.13 (Pin_13)
- net GPIO_41: now also J8.10 (Pin_10); no longer J8.16 (Pin_16)
- net GPIO_42: now also J8.12 (Pin_12); no longer J8.15 (Pin_15)
- net GPIO_43: now also J8.14 (Pin_14); no longer J8.18 (Pin_18)
- net GPIO_44: now also J8.16 (Pin_16); no longer J8.17 (Pin_17)
- net GPIO_48: now also J8.18 (Pin_18); no longer J8.19 (Pin_19)
- net VDD: now also Q1.3 (D), R8.2; no longer Q1.2 (S)
- net boot: now also R20.2
- net charger_out: now also Q1.2 (S); no longer Q1.3 (D)
- net at R11.1, SW4.2 (B): now also R7.2; no longer R10.2
- net GPIO_15 renamed bat_level
- net bat_level: now also R10.2, R8.1
Other:
- note added: "Battery level indicator"
- moved on the sheet: C13, C14, Q1, R11, R17, SW1, SW2, SW4A
