Commit message: Regenerated urdf from onshape model

File: SOFTWARE/little_red_rover_ws/src/little_red_rover/description/rover/robot.urdf (robot description, URDF)
Before this commit: robot little red rover, 4 links, 3 joints
Links:
- removed link wheel
- removed link wheel_2
- added link lidar_frame, mass 1e-9
- added link wheel_left, mass 0.060316879417403129748; collision mesh filename=http://localhost:8100/wheel_left.stl; visual mesh filename=http://localhost:8100/wheel_left_visual.stl
- added link wheel_right, mass 0.060316879417403573838; collision mesh filename=http://localhost:8100/wheel_right.stl; visual mesh filename=http://localhost:8100/wheel_right_visual.stl
- link robot_body: mass 0.19676137874980109688 -> 0.19785237681803841125
Joints:
- added joint lidar_frame_frame: type fixed, parent robot_body, child lidar_frame, origin xyz=-0.086199999999999873945 -3.4694469519536141888e-17 0.020785000000000775078 rpy=-4.5796699765786721216e-16 2.3850716431291444726e-30 3.9101198111849427206e-30, axis 0 0 0
- joint wheel_left_speed: child wheel_2 -> wheel_left; origin xyz=-0.011199999999997016162 0.043299999999999880251 -0.011370000000000322557 rpy=1.5707963267948970021 -2.2261824227171183414e-30 3.141592653589793116 -> xyz=-0.011199999999997394332 -0.043149999999999869016 -0.011369999999999999898 rpy=-1.570796326794896558 1.5707963267948594765 0
- joint wheel_right_speed: child wheel -> wheel_right; origin xyz=-0.011199999999997394332 -0.043149999999999869016 -0.011370000000000001633 rpy=-1.570796326794896558 -1.570796326794896336 0 -> xyz=-0.011199999999997014427 0.043299999999999880251 -0.011370000000000322557 rpy=-1.57079632679489678 5.4123372450415540448e-16 -3.141592653589793116

Commit message: Update robot URDF from onshape

File: SOFTWARE/little_red_rover_ws/src/little_red_rover/description/rover/robot.urdf (robot description, URDF)
Before this commit: robot little red rover, 5 links, 4 joints
Links:
- link wheel_left: mass 0.060316879417403129748 -> 0.060316879417403136687
- link wheel_right: mass 0.060316879417403573838 -> 0.06031687941740355996
Joints:
- joint lidar_frame_frame: origin xyz=-0.086199999999999873945 -3.4694469519536141888e-17 0.020785000000000775078 rpy=-4.5796699765786721216e-16 2.3850716431291444726e-30 3.9101198111849427206e-30 -> xyz=-0.086199999999999873945 -3.2250660475519238453e-17 0.020785000000000775078 rpy=-4.5796699765786721216e-16 2.3850716431291444726e-30 3.9101198111849427206e-30
- joint wheel_left_speed: origin xyz=-0.011199999999997394332 -0.043149999999999869016 -0.011369999999999999898 rpy=-1.570796326794896558 1.5707963267948594765 0 -> xyz=-0.011199999999997394332 -0.043149999999999820444 -0.011370000000000001633 rpy=-1.570796326794896558 1.570796326794896336 0
- joint wheel_right_speed: origin xyz=-0.011199999999997014427 0.043299999999999880251 -0.011370000000000322557 rpy=-1.57079632679489678 5.4123372450415540448e-16 -3.141592653589793116 -> xyz=-0.011199999999997014427 0.043299999999999880251 -0.011370000000000320822 rpy=1.5707963267948972241 -5.5511151231257728414e-17 -3.141592653589793116

Commit message: Invert lidar frame, fix agent disconnect causing a crash

File: SOFTWARE/little_red_rover_ws/src/little_red_rover/description/rover/robot.urdf (robot description, URDF)
Before this commit: robot little red rover, 5 links, 4 joints
Links:
- link robot_body: mass 0.19785237681803841125 -> 0.19785237681803843901
Joints:
- joint lidar_frame_frame: origin xyz=-0.086199999999999873945 -3.2250660475519238453e-17 0.020785000000000775078 rpy=-4.5796699765786721216e-16 2.3850716431291444726e-30 3.9101198111849427206e-30 -> xyz=-0.086199999999999873945 -3.2250660475519238453e-17 0.020785000000000771608 rpy=3.141592653589793116 -2.8726618518657236517e-44 2.9952754674941379765e-43
- joint wheel_left_speed: origin xyz=-0.011199999999997394332 -0.043149999999999820444 -0.011370000000000001633 rpy=-1.570796326794896558 1.570796326794896336 0 -> xyz=-0.011199999999997394332 -0.043149999999999869016 -0.011370000000000001633 rpy=-1.570796326794896558 7.7715611723761046577e-16 -6.4094948549207279255e-31

Commit message: PID control

File: SOFTWARE/little_red_rover_ws/src/little_red_rover/description/rover/robot.urdf (robot description, URDF)
Before this commit: robot little red rover, 5 links, 4 joints
Links:
- link robot_body: mass 0.19785237681803843901 -> 0.19763701795321664267
- link wheel_right: mass 0.06031687941740355996 -> 0.060316879417403580776

Commit message: Move foxglove bridge into ros2_workspace docker image, remove urdf server

File: SOFTWARE/little_red_rover_ws/src/little_red_rover/description/rover/robot.urdf (robot description, URDF)
Before this commit: robot little red rover, 5 links, 4 joints
Links:
- link robot_body: mass 0.19763701795321664267 -> 0.20115864605429473189; geometry collision mesh filename=package://little_red_rover/description/rover/lidar_motor.stl; collision mesh filename=package://little_red_rover/description/rover/lidar_top.stl
- link wheel_left: mass 0.060316879417403136687 -> 0.060316879417403129748; geometry collision mesh filename=package://little_red_rover/description/rover/wheel_left.stl; visual mesh filename=package://little_red_rover/description/rover/wheel_left_vis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
- link wheel_right: mass 0.060316879417403580776 -> 0.06031687941740355996; geometry collision mesh filename=package://little_red_rover/description/rover/wheel_right.stl; visual mesh filename=package://little_red_rover/description/rover/wheel_right_vi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
Joints:
- joint lidar_frame_frame: origin xyz=-0.086199999999999873945 -3.2250660475519238453e-17 0.020785000000000771608 rpy=3.141592653589793116 -2.8726618518657236517e-44 2.9952754674941379765e-43 -> xyz=-0.086199999999998278 -0.00024999999999992080424 0.023715000000000173441 rpy=3.1415926535897926719 1.0581813203458726654e-16 -9.1593399531631443431e-16
- joint wheel_left_speed: origin xyz=-0.011199999999997394332 -0.043149999999999869016 -0.011370000000000001633 rpy=-1.570796326794896558 7.7715611723761046577e-16 -6.4094948549207279255e-31 -> xyz=-0.011199999999998485473 -0.042049999999999934652 -0.011369999999999819487 rpy=1.5707963267948976682 -1.6601303665098055726e-15 -3.141592653589793116
- joint wheel_right_speed: origin xyz=-0.011199999999997014427 0.043299999999999880251 -0.011370000000000320822 rpy=1.5707963267948972241 -5.5511151231257728414e-17 -3.141592653589793116 -> xyz=-0.011199999999998036179 0.041550000000000003597 -0.011370000000000123064 rpy=-1.5707963267948956698 -8.3266726846886296798e-16 -1.3600232051663792198e-15

Commit message: Update robot description for proper wheel directions

File: SOFTWARE/little_red_rover_ws/src/little_red_rover/description/rover/robot.urdf (robot description, URDF)
Before this commit: robot little red rover, 5 links, 4 joints
Joints:
- removed joint wheel_left_speed
- removed joint wheel_right_speed
- added joint wheel_left: type continuous, parent robot_body, child wheel_left, origin xyz=-0.011199999999998485473 -0.042049999999999934652 -0.011369999999999819487 rpy=-1.5707963267948954478 -1.6601303665098055726e-15 -3.141592653589793116, axis 0 0 1, limit effort=1 velocity=20
- added joint wheel_right: type continuous, parent robot_body, child wheel_right, origin xyz=-0.011199999999998036179 0.041550000000000003597 -0.011370000000000123064 rpy=-1.5707963267948956698 -8.3266726846886296798e-16 -1.3600232051663792198e-15, axis 0 0 1, limit effort=1 velocity=20

Commit message: Wheel encoder only localization working

File: SOFTWARE/little_red_rover_ws/src/little_red_rover/description/rover/robot.urdf (robot description, URDF)
Before this commit: robot little red rover, 5 links, 4 joints
Links:
- removed link lidar_frame
- added link lidar, mass 1e-9
- link wheel_left: mass 0.060316879417403129748 -> 0.060316879417403122809
- link wheel_right: mass 0.06031687941740355996 -> 0.060316879417403553021
Joints:
- removed joint lidar_frame_frame
- added joint lidar_frame: type fixed, parent robot_body, child lidar, origin xyz=0.086200000000000123745 -1.3877787807814456755e-17 0.021884999999999994735 rpy=-3.141592653589793116 -3.2417252823925967892e-30 -3.141592653589793116, axis 0 0 0
- joint wheel_left: origin xyz=-0.011199999999998485473 -0.042049999999999934652 -0.011369999999999819487 rpy=-1.5707963267948954478 -1.6601303665098055726e-15 -3.141592653589793116 -> xyz=0.011199999999999927028 0.041799999999999955247 -0.013199999999999987785 rpy=-1.5707963267948970021 2.7802557667454690514e-14 -6.5919492087118866803e-16
- joint wheel_right: origin xyz=-0.011199999999998036179 0.041550000000000003597 -0.011370000000000123064 rpy=-1.5707963267948956698 -8.3266726846886296798e-16 -1.3600232051663792198e-15 -> xyz=0.01119999999999957141 -0.041800000000000038514 -0.013200000000000263606 rpy=-1.5707963267948961139 6.257321276414477704e-14 3.1415926535897926719

Commit message: Update URDF to match CAD

File: SOFTWARE/little_red_rover_ws/src/little_red_rover/description/rover/robot.urdf (robot description, URDF)
Before this commit: robot little red rover, 5 links, 4 joints
Links:
- added link base_footprint, mass 1e-9
- link wheel_left: mass 0.060316879417403122809 -> 0.060316879417403136687
- link wheel_right: mass 0.060316879417403553021 -> 0.06031687941740355996
Joints:
- added joint base_footprint_frame: type fixed, parent robot_body, child base_footprint, origin xyz=0.011199999999999710187 0 -0.043680000000000086813 rpy=-5.9164567891575902922e-31 -6.1629758220391558245e-32 4.8461212225578935465e-32, axis 0 0 0
